File: PCB/PCB.kicad_pcb (KiCad board)
At the start: 2 copper layers, 418.3 x 124.6 mm, 423 parts, among them J2 Conn_OLED_I2C, U1 74AHCT125

Commit message: updated the PCB a little bit
Parts:
- added C105: 100nF, Capacitor_SMD:C_0805_2012Metric_Pad1.18x1.45mm_HandSolder, F.Cu at (88.3, 148.7)
Connections:
- U1 pad 12: unconnected-(U1-Pad12) -> GND
- U1 pad 5: unconnected-(U1-Pad5) -> GND
- U1 pad 9: unconnected-(U1-Pad9) -> GND
Routing:
- net +3V3: track 29.3 -> 31.4 mm
- net Net-(D155-DOUT): track 26.2 -> 26.9 mm
- net GND: vias 398 -> 427
- net (no net): vias 12 -> 5
