File: PCB/PCB.kicad_pcb (KiCad board)
At the start: 2 copper layers, 418.3 x 124.6 mm, 424 parts, among them J2 Conn_OLED_I2C, U1 74AHCT125

Commit message: updated screw holes on the PCB
Other:
- outline, holes or cut-outs redrawn
- board text added: "YD-RP2040"
Changed lines of the file:
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@@
 	(gr_circle
 		(center 71.6105 256.9272)
-		(end 77.0105 256.9272)
+		(end 74.5105 256.9272)
 		(stroke
 			(width 0.1)
@@
 	(gr_circle
 		(center 401.7897 194.9438)
-		(end 407.1897 194.9438)
+		(end 404.6897 194.9438)
 		(stroke
 			(width 0.1)
@@
 	(gr_circle
 		(center 101.1333 210.0241)
-		(end 106.5333 210.0241)
+		(end 104.0333 210.0241)
 		(stroke
 			(width 0.1)
@@
 	(gr_circle
 		(center 478.839084 256.8524)
-		(end 484.239084 256.8524)
+		(end 481.739084 256.8524)
 		(stroke
 			(width 0.05)
@@
 	(gr_circle
 		(center 71.6105 256.9272)
-		(end 74.7105 256.9272)
+		(end 73.1605 256.9272)
 		(stroke
 			(width 0.05)
@@
 	(gr_circle
 		(center 401.7897 194.9438)
-		(end 404.8897 194.9438)
+		(end 403.3397 194.9438)
 		(stroke
 			(width 0.05)
@@
 	(gr_circle
 		(center 101.0522 210.0241)
-		(end 104.1522 210.0241)
+		(end 102.6022 210.0241)
 		(stroke
 			(width 0.05)
@@
 	(gr_circle
 		(center 478.8534 256.8524)
-		(end 481.9534 256.8524)
+		(end 480.4034 256.8524)
 		(stroke
 			(width 0.05)
@@
 		)
 	)
+	(gr_text "YD-RP2040"
+		(at 103.906832 161.364433 90)
+		(layer "B.SilkS")
+		(effects
+			(font
+				(size 1.5 1.5)
+				(thickness 0.3)
+				(bold yes)
+			)
+			(justify left bottom mirror)
+		)
+	)
 	(via
 		(at 444.6495 251.2965)
@@
 	)
 	(segment
-		(start 104.1522 171.1328)
-		(end 104.9459 171.9265)
+		(start 104.9459 171.9265)
+		(end 104.9459 187.0068)
 		(width 0.2)
 		(layer "F.Cu")
@@
 	)
 	(segment
-		(start 111.2955 207.9926)
-		(end 106.5333 212.7548)
+		(start 105.7396 162.4021)
+		(end 97.8026 170.3391)
 		(width 0.2)
 		(layer "F.Cu")
@@
 	)
 	(segment
-		(start 105.7396 162.4021)
-		(end 97.8026 170.3391)
+		(start 390.6779 207.643)
+		(end 391.4716 208.4367)
 		(width 0.2)
 		(layer "F.Cu")
@@
 	)
 	(segment
-		(start 390.6779 207.643)
-		(end 391.4716 208.4367)
+		(start 111.2955 193.3564)
+		(end 111.2955 207.9926)
 		(width 0.2)
 		(layer "F.Cu")
@@
 	)
 	(segment
-		(start 106.5333 212.7548)
-		(end 106.5333 213.5485)
+		(start 104.9459 187.0068)
+		(end 111.2955 193.3564)
 		(width 0.2)
 		(layer "F.Cu")
@@
 	)
 	(segment
-		(start 104.9459 171.9265)
-		(end 104.9459 187.0068)
+		(start 104.3715 171.3521)
+		(end 104.9459 171.9265)
 		(width 0.2)
 		(layer "F.Cu")
@@
 	)
 	(segment
-		(start 104.9459 187.0068)
-		(end 111.2955 193.3564)
+		(start 111.2955 207.9926)
+		(end 106.5333 212.7548)
 		(width 0.2)
 		(layer "F.Cu")
@@
 	)
 	(segment
+		(start 106.5333 212.7548)
+		(end 106.5333 213.5485)
+		(width 0.2)
+		(layer "F.Cu")
+		(net 140)
+	)
+	(segment
 		(start 106.5333 221.4855)
 		(end 106.5333 217.517)
@@
 	)
 	(segment
-		(start 111.2955 193.3564)
-		(end 111.2955 207.9926)
-		(width 0.2)
-		(layer "F.Cu")
-		(net 140)
-	)
-	(segment
 		(start 375.5976 159.2273)
 		(end 372.4228 162.4021)
@@
 	)
 	(via
-		(at 104.1522 171.1328)
+		(at 104.3715 171.3521)
 		(size 0.7)
 		(drill 0.3)
@@
 	)
 	(segment
-		(start 103.3585 170.3391)
-		(end 97.8026 170.3391)
-		(width 0.2)
-		(layer "B.Cu")
-		(net 140)
-	)
-	(segment
 		(start 412.9015 187.0068)
 		(end 451.8922 187.0068)
@@
 	)
 	(segment
-		(start 370.0417 162.4021)
-		(end 347.8181 162.4021)
+		(start 104.3715 171.3521)
+		(end 103.3585 170.3391)
 		(width 0.2)
 		(layer "B.Cu")
@@
 	)
 	(segment
-		(start 104.1522 171.1328)
-		(end 103.3585 170.3391)
+		(start 370.0417 162.4021)
+		(end 347.8181 162.4021)
 		(width 0.2)
 		(layer "B.Cu")
@@
 		(width 0.2)
 		(layer "B.Cu")
+		(net 140)
+	)
+	(segment
+		(start 103.3585 170.3391)
+		(end 97.8026 170.3391)
+		(width 0.2)
+		(layer "B.Cu")
